Commit message: rotated the body to match the coordinate system

File: src/open_mower/urdf/yardforce-sc600eco.urdf (robot description, URDF)
Before this commit: robot open_mower, 3 links, 2 joints
Links:
- link base_link: geometry visual box size=0.54 0.34 0.20
Joints:
- joint bumper_left_joint: origin xyz=-0.17 0.54 0.040 rpy=0 0 0 -> xyz=0.40 0.17 0.040 rpy=0 0 0
- joint bumper_right_joint: origin xyz=-0.17 0.54 0.040 rpy=0 0 0 -> xyz=0.40 -0.17 0.040 rpy=0 0 0

Commit message: testing

File: src/open_mower/urdf/yardforce-sc600eco.urdf (robot description, URDF)
Before this commit: robot open_mower, 3 links, 2 joints
Links:
- added link base_footprint
- link base_link: geometry 
Joints:
- added joint base_link_joint: type fixed, parent base_footprint, child base_link, origin xyz=0 0 0.08 rpy=0 0 0
